File: doc/schematics_kicad/kicad/tenacle_MCU_PYBV11.kicad_sch (KiCad schematic)
At the start: 3 parts, among them T301 tentacle_octobus, T302 tentacle_relay

Commit message: MCU names as in micropython-git
Other:
- sheet pyboard3 renamed MCU_PYBV11
- sheet MCU_PYBV11: file mcu_pyboard.kicad_sch -> mcu_PYBV11.kicad_sch
- title: tentacle_MCU_grobotics_pyboard -> tentacle_MCU_PYBV11
Changed lines of the file:
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@@
 	(paper "A4")
 	(title_block
-		(title "tentacle_MCU_grobotics_pyboard")
+		(title "tentacle_MCU_PYBV11")
 		(date "2024-07-16")
 		(company "Hans Märki, Märki Informatik")
@@
 			(color 0 0 0 0.0000)
 		)
-		(property "Sheetname" "pyboard3"
+		(property "Sheetname" "MCU_PYBV11"
 			(at 179.07 46.2784 0)
 			(effects
@@
 			)
 		)
-		(property "Sheetfile" "mcu_pyboard.kicad_sch"
+		(property "Sheetfile" "mcu_PYBV11.kicad_sch"
 			(at 179.07 100.9146 0)
 			(effects
